File: hardware/cart/hw/wallet/GameboyCartridgeV2.1.kicad_pcb (KiCad board)
At the start: 6 copper layers, 52.8 x 61.2 mm, 146 parts, among them J1 USB_C_Receptacle_USB2.0, J2 Micro_SD_Card_Det2, J4 Conn_01x06, J5 CartBus, Q1 CJ2302, Q101 SIA975DJ-T1-GE3, Q102 2N7002, SW1 SW_Push, SW2 SW_Push, U1 USBLC6-2P6, U101 TPS2116DRLR, U102 TPS2553DBVR, U103 TPS63802DLAR, U104 ESP32-C3-MINI-1U-N4, U105 SN74LVC1G125DBVR, U106 SN74LVC3G34DCTR, U107 CH334P, U108 TLV3012BIDBVR, U109 TLV431BIDBZR, U2 W25Q128JVSIQ, U3 RP2350_80QFN, U4 IS66WVH8M8BLL-100B1LI, U5 MCP79510, U6 AP2112K-3.3, U7 TXB0108PW, Y1 12MHz, Y101 12MHz 10pF 10ppm, Y2 32.768kHz

Commit message: hardware/cart: wallet variant of the WiFi cart board (SE050E2 + LIS3DH)
Removes HyperRAM, microSD and RTC (DNP, off board). Adds the NXP SE050E2
secure element on I2C1 (GPIO6/7, ENA GPIO10, Deep Power-down wiring) and a
LIS3DH on I2C0 (GPIO8/9, INT1 GPIO11) in the freed area, placed and routed.
SE050 footprint generated from NXP SOT1969-1; JLC's footprint confirms it.

Gates: kicad_check (ERC/DRC 0 new, 0 unconnected, parity clean),
netlist_check, design_calcs, sim_vs_netlist all PASS. BOM: 1 FAIL, L1
(Croco's RP2350 inductor) out of stock, left for review. Not ready to order.

Co-Authored-By: Claude Opus 5.5 (1M context) <noreply@anthropic.com>
Claude-Session: https://claude.ai/code/session_01K3DS9Lp5DvbMPN1T6z91y9
Parts:
- removed C22, C23, C24: 100nF, Capacitor_SMD:C_0603_1608Metric
- removed C27, C28: 4.3pF, Capacitor_SMD:C_0603_1608Metric
- removed J2: Micro_SD_Card_Det2, Connector_Card:microSD_HC_Hirose_DM3D-SF
- removed R12, R15, R17, R6: 10k, Resistor_SMD:R_0603_1608Metric
- removed TP1, TP2, TP3, TP4: TestPoint, TestPoint:TestPoint_Pad_D1.0mm
- removed U4: IS66WVH8M8BLL-100B1LI, CrocoV2:BGA25C100P5X5_800X600X120N
- removed U5: MCP79510, Package_SO:MSOP-10_3x3mm_P0.5mm
- removed Y2: 32.768kHz, Crystal:Crystal_SMD_TXC_9HT11-2Pin_2.0x1.2mm
- added C125: 100nF 16V X7R, Capacitor_SMD:C_0402_1005Metric, F.Cu at (136.9, 94.4)
- added C126: 100nF 16V X7R, Capacitor_SMD:C_0402_1005Metric, F.Cu at (134.2, 91.3)
- added C127: 100nF 16V X7R, Capacitor_SMD:C_0402_1005Metric, F.Cu at (130.2, 91.7)
- added C128: 10uF 10V X5R, Capacitor_SMD:C_0603_1608Metric, F.Cu at (127.7, 94.0)
- added R133: 2.2k, Resistor_SMD:R_0402_1005Metric, F.Cu at (134.7, 97.2)
- added R134: 2.2k, Resistor_SMD:R_0402_1005Metric, F.Cu at (135.7, 97.2)
- added R135: 100k, Resistor_SMD:R_0402_1005Metric, F.Cu at (136.9, 96.6)
- added R136: 4.7k, Resistor_SMD:R_0402_1005Metric, F.Cu at (129.8, 97.2)
- added R137: 4.7k, Resistor_SMD:R_0402_1005Metric, F.Cu at (130.8, 97.2)
- added U110: SE050E2HQ1/Z01Z3Z, radio:NXP_HX2QFN-20-1EP_3x3mm_P0.4mm_EP1.9x1.9mm, F.Cu at (134.2, 94.0)
- added U111: LIS3DHTR, Package_LGA:LGA-16_3x3mm_P0.5mm_LayoutBorder3x5y, F.Cu at (130.2, 94.0)
Connections:
- U3 pad 3: HYPERRAM_RWDS -> SE_SDA
- U3 pad 4: HYPERRAM_CLK -> SE_SCL
- U3 pad 6: HYPERRAM_CS -> ACC_SDA
- U3 pad 7: /CPU/HYPERRAM_DQ0 -> ACC_SCL
- U3 pad 8: /CPU/HYPERRAM_DQ1 -> SE_ENA
- U3 pad 9: /CPU/HYPERRAM_DQ2 -> ACC_INT1
Routing:
- net RTC_CS: track 44.0 -> 0.00 mm, vias 3 -> 0
- net SD_CARD_CS: track 30.0 -> 0.00 mm, vias 2 -> 0
- net GND: track 272.2 -> 242.8 mm, vias 214 -> 219
- net HYPERRAM_CS: track 26.9 -> 0.00 mm, vias 2 -> 0
- net /CPU/HYPERRAM_DQ4: track 21.0 -> 0.00 mm
- net /CPU/HYPERRAM_DQ7: track 21.0 -> 0.00 mm
- net /CPU/HYPERRAM_DQ3: track 21.0 -> 0.00 mm
- net /CPU/HYPERRAM_DQ2: track 20.9 -> 0.00 mm
- net ACC_SDA: track 0.00 -> 20.7 mm, vias 0 -> 2
- net HYPERRAM_RWDS: track 19.7 -> 0.00 mm, vias 2 -> 0
- net HYPERRAM_CLK: track 19.7 -> 0.00 mm, vias 2 -> 0
- net /CPU/HYPERRAM_DQ0: track 19.7 -> 0.00 mm, vias 2 -> 0
- net /CPU/HYPERRAM_DQ6: track 19.6 -> 0.00 mm, vias 2 -> 0
- net /CPU/HYPERRAM_DQ5: track 19.5 -> 0.00 mm, vias 2 -> 0
- net /CPU/HYPERRAM_DQ1: track 19.5 -> 0.00 mm, vias 2 -> 0
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