File: hardware/cart/hw/wallet/GameboyCartridgeV2.1.kicad_pcb (KiCad board)
At the start: 6 copper layers, 52.8 x 61.2 mm, 140 parts, among them J1 USB_C_Receptacle_USB2.0, J4 Conn_01x06, J5 CartBus, Q1 CJ2302, Q101 SIA975DJ-T1-GE3, Q102 2N7002, SW1 SW_Push, SW2 SW_Push, U1 USBLC6-2P6, U101 TPS2116DRLR, U102 TPS2553DBVR, U103 TPS63802DLAR, U104 ESP32-C3-MINI-1U-N4, U105 SN74LVC1G125DBVR, U106 SN74LVC3G34DCTR, U107 CH334P, U108 TLV3012BIDBVR, U109 TLV431BIDBZR, U110 SE050E2HQ1/Z01Z3Z, U111 LIS3DHTR, U2 W25Q128JVSIQ, U3 RP2350_80QFN, U6 AP2112K-3.3, U7 TXB0108PW, Y1 12MHz, Y101 12MHz 10pF 10ppm

Commit message: Cartridge board: full checks and simulations, routing polish, kagiboy back silk
- Power stage audits on this board with vendor SPICE models: A1-A7 81 PASS,
  A8 114 PASS (radio power manager C code and .spiceinit brought along).
- Bus simulation with the real ROM: TXB0108 @150 MHz, 81.8 ns margin, 0 errors.
- design_calcs: I2C sections for the SE050 (Fm+) and LIS3DH (Fm) buses.
- Routing cleaned (121 router segments removed, collinear pairs merged),
  no stubs or dangling copper.
- Back silkscreen: kagiboy logo, wallet label, github.com/hazy2go/kagiboy.
- SE050 3D model for renders; height check uses the datasheet height.
- L1 kept (RP2350 datasheet requires the polarity-marked part); out of
  stock at JLC, hold until restock or pre-order.
- README: dated Updates section with board images; docs/hardware.md points
  to the board.

All gates PASS (ERC/DRC 0 new, unconnected 0, parity, netlist, calcs,
sim-vs-netlist, height); ROM build, tsc, web build, smoke PASS.

Co-Authored-By: Claude Opus 5.5 (1M context) <noreply@anthropic.com>
Claude-Session: https://claude.ai/code/session_01K3DS9Lp5DvbMPN1T6z91y9
Routing:
- net /Radio/ADC_VCC: track 28.8 -> 28.0 mm
Other:
- board text added: "github.com/hazy2go/kagiboy"
- board text added: "kagiboy wallet Rev A 10/2026 RP2350B+SE050E2"
- board text removed: "RemAI"
- board text removed: "WiFi Cartridge Rev B 10/2026 RP2350B+ESP32C3"
- board text removed: "co-created with"
- board text removed: "github.com/hazy2go/wifi-game-boy-cartridge"

Commit message: Cartridge board: kagiboy-only branding, wallet order sheet, Gerber zip
Back silkscreen no longer carries the base-design credit (it lives in the
WiFi cart repo); licence file and source notices kept per CERN-OHL-P.
ORDER.md rewritten for the wallet board. Gerbers regenerated and zipped.
Gate PASS (ERC/DRC 0 new, unconnected 0, parity).

Co-Authored-By: Claude Opus 5.5 (1M context) <noreply@anthropic.com>
Claude-Session: https://claude.ai/code/session_01K3DS9Lp5DvbMPN1T6z91y9
Other:
- board text removed: "based on Croco Cartridge V2.1 by shilga"
Changed lines of the file:
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@@
-		)
-	)
-	(gr_text "based on Croco Cartridge\nV2.1 by shilga"
-		(at 135.3 108.4 0)
-		(layer "B.SilkS")
-		(effects
-			(font
-				(size 0.8 0.8)
-				(thickness 0.15)
-			)
-			(justify left bottom mirror)
 		)
 	)
