File: hardware/cart/hw/wallet/GameboyCartridgeV2.1.kicad_pcb (KiCad board)
At the start: 6 copper layers, 52.8 x 61.2 mm, 140 parts, among them J1 USB_C_Receptacle_USB2.0, J4 Conn_01x06, J5 CartBus, Q1 CJ2302, Q101 SIA975DJ-T1-GE3, Q102 2N7002, SW1 SW_Push, SW2 SW_Push, U1 USBLC6-2P6, U101 TPS2116DRLR, U102 TPS2553DBVR, U103 TPS63802DLAR, U104 ESP32-C3-MINI-1U-N4, U105 SN74LVC1G125DBVR, U106 SN74LVC3G34DCTR, U107 CH334P, U108 TLV3012BIDBVR, U109 TLV431BIDBZR, U110 SE050E2HQ1/Z01Z3Z, U111 LIS3DHTR, U2 W25Q128JVSIQ, U3 RP2350_80QFN, U6 AP2112K-3.3, U7 TXB0108PW, Y1 12MHz, Y101 12MHz 10pF 10ppm

Commit message: Board: fixes from an independent datasheet review (2026-10-16)
A fresh reviewer, without our notes or gates, checked the schematic and board
against every datasheet. Fixed:
- radio-area ground: F.Cu pour, 60 stitching vias, 9 vias in the ESP32-C3
  centre pad, vias at the TPS63802 GND pins (219 -> 296 GND vias)
- VREG_LX cut-out on In1-In4 (RP2350 DS 6.3.8, Fig. 27); ESP CS and LED_DIN
  re-routed around it
- R110 91k: C4147 (below JLC minimum buy) -> C453777
- R138 4.7k pull-down on the TXB0108 OE (SCES643 sec 9)
- Y1: ABM8-272-T3 (C20625731), the crystal Raspberry Pi specifies
- USB upstream pair: both lines on In2 over solid ground, 2 vias each

Kept, with reasons in the LOGBOOK: radio input threshold, D1 on 3V3, antenna.
All gates, power audits (81/114) and fab outputs re-run. New tools:
add_pour, gnd_stitch, lx_keepout, inner_link.

Co-Authored-By: Claude Opus 5.5 (1M context) <noreply@anthropic.com>
Claude-Session: https://claude.ai/code/session_01K3DS9Lp5DvbMPN1T6z91y9
Parts:
- added R138: 4.7k, Resistor_SMD:R_0402_1005Metric, F.Cu at (149.8, 105.0)
Routing:
- net DEBUG_UART_TX: track 54.0 -> 61.8 mm
- net GND: track 242.8 -> 245.8 mm, vias 219 -> 296
- net USB_D_prot+: track 14.2 -> 12.4 mm, vias 3 -> 2
- net LED_DIN: track 18.5 -> 19.9 mm
- net GBBUS_EN: track 17.2 -> 18.6 mm
