File: hardware/cart/hw/wallet/cpu.kicad_sch (KiCad schematic)
At the start: 61 parts, among them J1 USB_C_Receptacle_USB2.0, J2 Micro_SD_Card_Det2, J3 DBG_UART, J4 Conn_01x06, SW1 SW_Push, SW2 SW_Push, U1 USBLC6-2P6, U2 W25Q128JVSIQ, U3 RP2350_80QFN, U4 IS66WVH8M8BLL-100B1LI, U5 MCP79510, Y1 12MHz, Y2 32.768kHz

Commit message: hardware/cart: wallet variant of the WiFi cart board (SE050E2 + LIS3DH)
Removes HyperRAM, microSD and RTC (DNP, off board). Adds the NXP SE050E2
secure element on I2C1 (GPIO6/7, ENA GPIO10, Deep Power-down wiring) and a
LIS3DH on I2C0 (GPIO8/9, INT1 GPIO11) in the freed area, placed and routed.
SE050 footprint generated from NXP SOT1969-1; JLC's footprint confirms it.

Gates: kicad_check (ERC/DRC 0 new, 0 unconnected, parity clean),
netlist_check, design_calcs, sim_vs_netlist all PASS. BOM: 1 FAIL, L1
(Croco's RP2350 inductor) out of stock, left for review. Not ready to order.

Co-Authored-By: Claude Opus 5.5 (1M context) <noreply@anthropic.com>
Claude-Session: https://claude.ai/code/session_01K3DS9Lp5DvbMPN1T6z91y9
Parts:
- C22, C23, C24, C27, C28, J2, R12, R15, R6, U4, U5, Y2: now not fitted; now left out of the parts list
- R17: now left out of the parts list
- TP1, TP2, TP3, TP4: now not fitted
Connections:
- net HYPERRAM_CLK: no longer U3.4 (GPIO7)
- net HYPERRAM_CS: no longer U3.6 (GPIO8)
- net HYPERRAM_DQ0: no longer U3.7 (GPIO9)
- net HYPERRAM_DQ1: no longer U3.8 (GPIO10)
- net HYPERRAM_DQ2: no longer U3.9 (GPIO11)
- net HYPERRAM_RWDS: no longer U3.3 (GPIO6)
- new net ACC_INT1: U3.9 (GPIO11)
- new net ACC_SCL: U3.7 (GPIO9)
- new net ACC_SDA: U3.6 (GPIO8)
- new net SE_ENA: U3.8 (GPIO10)
- new net SE_SCL: U3.4 (GPIO7)
- new net SE_SDA: U3.3 (GPIO6)
Changed lines of the file:
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@@
 	)
 	(bus_entry
-		(at 266.7 107.95)
-		(size 2.54 2.54)
-		(stroke
-			(width 0)
-			(type default)
-		)
-	)
-	(bus_entry
 		(at 246.38 135.89)
 		(size 2.54 2.54)
@@
 	)
 	(bus_entry
-		(at 266.7 110.49)
-		(size 2.54 2.54)
-		(stroke
-			(width 0)
-			(type default)
-		)
-	)
-	(bus_entry
 		(at 246.38 148.59)
 		(size 2.54 2.54)
@@
 	)
 	(bus_entry
-		(at 266.7 113.03)
-		(size 2.54 2.54)
-		(stroke
-			(width 0)
-			(type default)
-		)
-	)
-	(bus_entry
 		(at 227.33 262.89)
 		(size 2.54 2.54)
@@
 	(wire
 		(pts
-			(xy 233.68 107.95) (xy 266.7 107.95)
-		)
-		(stroke
-			(width 0)
-			(type default)
-		)
-	)
-	(wire
-		(pts
 			(xy 387.35 149.86) (xy 387.35 151.13)
 		)
@@
 	(wire
 		(pts
-			(xy 233.68 110.49) (xy 266.7 110.49)
-		)
-		(stroke
-			(width 0)
-			(type default)
-		)
-	)
-	(wire
-		(pts
 			(xy 203.2 275.59) (xy 200.66 275.59)
 		)
@@
 		)
 	)
-	(wire
-		(pts
-			(xy 233.68 113.03) (xy 266.7 113.03)
-		)
-		(stroke
-			(width 0)
-			(type default)
-		)
-	)
 	(bus
 		(pts
@@
 		)
 	)
-	(label "HYPERRAM_DQ1"
-		(at 250.19 110.49 0)
-		(effects
-			(font
-				(size 1.27 1.27)
-			)
-			(justify left bottom)
-		)
-	)
-	(label "HYPERRAM_DQ2"
-		(at 250.19 113.03 0)
-		(effects
-			(font
-				(size 1.27 1.27)
-			)
-			(justify left bottom)
-		)
-	)
 	(label "FLASH_SS"
 		(at 43.18 167.64 0)
@@
 		)
 	)
-	(label "HYPERRAM_DQ0"
-		(at 250.19 107.95 0)
-		(effects
-			(font
-				(size 1.27 1.27)
-			)
-			(justify left bottom)
-		)
-	)
 	(label "VBUS_raw"
 		(at 52.07 29.21 0)
@@
 		)
 	)
-	(global_label "HYPERRAM_CLK"
+	(global_label "SE_SCL"
 		(shape output)
 		(at 234.95 102.87 0)
@@
 		)
 	)
-	(global_label "HYPERRAM_CS"
+	(global_label "ACC_SDA"
 		(shape output)
 		(at 234.95 105.41 0)
@@
 		)
 	)
-	(global_label "HYPERRAM_RWDS"
+	(global_label "SE_SDA"
 		(shape bidirectional)
 		(at 234.95 100.33 0)
@@
 		(unit 1)
 		(exclude_from_sim no)
-		(in_bom yes)
-		(on_board yes)
-		(dnp no)
+		(in_bom no)
+		(on_board no)
+		(dnp yes)
 		(property "Reference" "R15"
 			(at 309.372 177.6984 0)
@@
 		(exclude_from_sim no)
 		(in_bom no)
-		(on_board yes)
-		(dnp no)
+		(on_board no)
+		(dnp yes)
 		(property "Reference" "TP2"
 			(at 183.642 272.288 0)
@@
 		(exclude_from_sim no)
 		(in_bom no)
-		(on_board yes)
-		(dnp no)
+		(on_board no)
+		(dnp yes)
 		(property "Reference" "TP1"
 			(at 292.862 206.502 0)
@@
 		(unit 1)
 		(exclude_from_sim no)
-		(in_bom yes)
-		(on_board yes)
-		(dnp no)
+		(in_bom no)
+		(on_board no)
+		(dnp yes)
 		(property "Reference" "C23"
 			(at 186.309 239.9284 0)
@@
 		(unit 1)
 		(exclude_from_sim no)
-		(in_bom yes)
-		(on_board yes)
-		(dnp no)
+		(in_bom no)
+		(on_board no)
+		(dnp yes)
 		(property "Reference" "C24"
 			(at 334.899 177.6984 0)
@@
 		(unit 1)
 		(exclude_from_sim no)
-		(in_bom yes)
-		(on_board yes)
+		(in_bom no)
+		(on_board no)
 		(dnp yes)
 		(property "Reference" "R17"
@@
 		(unit 1)
 		(exclude_from_sim no)
-		(in_bom yes)
-		(on_board yes)
-		(dnp no)
+		(in_bom no)
+		(on_board no)
+		(dnp yes)
 		(property "Reference" "R6"
 			(at 106.172 214.5284 0)
@@
 		(unit 1)
 		(exclude_from_sim no)
-		(in_bom yes)
-		(on_board yes)
-		(dnp no)
+		(in_bom no)
+		(on_board no)
+		(dnp yes)
 		(fields_autoplaced yes)
 		(property "Reference" "Y2"
@@
 		(exclude_from_sim no)
 		(in_bom no)
-		(on_board yes)
-		(dnp no)
+		(on_board no)
+		(dnp yes)
 		(property "Reference" "TP4"
 			(at 186.182 246.888 0)
@@
 		(exclude_from_sim no)
 		(in_bom no)
-		(on_board yes)
-		(dnp no)
+		(on_board no)
+		(dnp yes)
 		(property "Reference" "TP3"
 			(at 186.436 260.096 0)
@@
 		(unit 1)
 		(exclude_from_sim no)
-		(in_bom yes)
-		(on_board yes)
-		(dnp no)
+		(in_bom no)
+		(on_board no)
+		(dnp yes)
 		(property "Reference" "C27"
 			(at 345.5416 186.309 0)
@@
 		(unit 1)
 		(exclude_from_sim no)
-		(in_bom yes)
-		(on_board yes)
-		(dnp no)
+		(in_bom no)
+		(on_board no)
+		(dnp yes)
 		(fields_autoplaced yes)
 		(property "Reference" "J2"
@@
 		(unit 1)
 		(exclude_from_sim no)
-		(in_bom yes)
-		(on_board yes)
-		(dnp no)
+		(in_bom no)
+		(on_board no)
+		(dnp yes)
 		(property "Reference" "C22"
 			(at 173.609 239.9284 0)
@@
 		(unit 1)
 		(exclude_from_sim no)
-		(in_bom yes)
-		(on_board yes)
-		(dnp no)
+		(in_bom no)
+		(on_board no)
+		(dnp yes)
 		(property "Reference" "R12"
 			(at 156.972 252.6284 0)
@@
 		(unit 1)
 		(exclude_from_sim no)
-		(in_bom yes)
-		(on_board yes)
-		(dnp no)
+		(in_bom no)
+		(on_board no)
+		(dnp yes)
 		(property "Reference" "U4"
 			(at 205.2194 237.6002 0)
@@
 		(unit 1)
 		(exclude_from_sim no)
-		(in_bom yes)
-		(on_board yes)
-		(dnp no)
+		(in_bom no)
+		(on_board no)
+		(dnp yes)
 		(property "Reference" "C28"
 			(at 347.8784 201.041 0)
@@
 		(unit 1)
 		(exclude_from_sim no)
-		(in_bom yes)
-		(on_board yes)
-		(dnp no)
+		(in_bom no)
+		(on_board no)
+		(dnp yes)
 		(fields_autoplaced yes)
 		(property "Reference" "U5"
@@
 		)
 	)
-)
+	(global_label "ACC_SCL"
+		(shape bidirectional)
+		(at 233.68 107.95 0)
+		(fields_autoplaced yes)
+		(effects
+			(font
+				(size 1.27 1.27)
+			)
+			(justify left)
+		)
+	)
+	(global_label "SE_ENA"
+		(shape bidirectional)
+		(at 233.68 110.49 0)
+		(fields_autoplaced yes)
+		(effects
+			(font
+				(size 1.27 1.27)
+			)
+			(justify left)
+		)
+	)
+	(global_label "ACC_INT1"
+		(shape bidirectional)
+		(at 233.68 113.03 0)
+		(fields_autoplaced yes)
+		(effects
+			(font
+				(size 1.27 1.27)
+			)
+			(justify left)
+		)
+	))
