File: hardware/cart/hw/wallet/cpu.kicad_sch (KiCad schematic)
At the start: 61 parts, among them J1 USB_C_Receptacle_USB2.0, J2 Micro_SD_Card_Det2, J3 DBG_UART, J4 Conn_01x06, SW1 SW_Push, SW2 SW_Push, U1 USBLC6-2P6, U2 W25Q128JVSIQ, U3 RP2350_80QFN, U4 IS66WVH8M8BLL-100B1LI, U5 MCP79510, Y1 12MHz, Y2 32.768kHz

Commit message: Board: fixes from an independent datasheet review (2026-10-16)
A fresh reviewer, without our notes or gates, checked the schematic and board
against every datasheet. Fixed:
- radio-area ground: F.Cu pour, 60 stitching vias, 9 vias in the ESP32-C3
  centre pad, vias at the TPS63802 GND pins (219 -> 296 GND vias)
- VREG_LX cut-out on In1-In4 (RP2350 DS 6.3.8, Fig. 27); ESP CS and LED_DIN
  re-routed around it
- R110 91k: C4147 (below JLC minimum buy) -> C453777
- R138 4.7k pull-down on the TXB0108 OE (SCES643 sec 9)
- Y1: ABM8-272-T3 (C20625731), the crystal Raspberry Pi specifies
- USB upstream pair: both lines on In2 over solid ground, 2 vias each

Kept, with reasons in the LOGBOOK: radio input threshold, D1 on 3V3, antenna.
All gates, power audits (81/114) and fab outputs re-run. New tools:
add_pour, gnd_stitch, lx_keepout, inner_link.

Co-Authored-By: Claude Opus 5.5 (1M context) <noreply@anthropic.com>
Claude-Session: https://claude.ai/code/session_01K3DS9Lp5DvbMPN1T6z91y9
Parts:
- Y1: LCSC C668845 -> C20625731
Changed lines of the file:
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@@
 			)
 		)
-		(property "LCSC" "C668845"
+		(property "LCSC" "C20625731"
 			(at 148.59 125.73 90)
 			(effects
