File: hardware/cart/hw/wallet/radio.kicad_sch (KiCad schematic)
At the start: 70 parts, among them Q101 SIA975DJ-T1-GE3, Q102 2N7002, U101 TPS2116DRLR, U102 TPS2553DBVR, U103 TPS63802DLAR, U104 ESP32-C3-MINI-1U-N4, U105 SN74LVC1G125DBVR, U106 SN74LVC3G34DCTR, U107 CH334P, U108 TLV3012BIDBVR, U109 TLV431BIDBZR, Y101 12MHz 10pF 10ppm

Commit message: hardware/cart: wallet variant of the WiFi cart board (SE050E2 + LIS3DH)
Removes HyperRAM, microSD and RTC (DNP, off board). Adds the NXP SE050E2
secure element on I2C1 (GPIO6/7, ENA GPIO10, Deep Power-down wiring) and a
LIS3DH on I2C0 (GPIO8/9, INT1 GPIO11) in the freed area, placed and routed.
SE050 footprint generated from NXP SOT1969-1; JLC's footprint confirms it.

Gates: kicad_check (ERC/DRC 0 new, 0 unconnected, parity clean),
netlist_check, design_calcs, sim_vs_netlist all PASS. BOM: 1 FAIL, L1
(Croco's RP2350 inductor) out of stock, left for review. Not ready to order.

Co-Authored-By: Claude Opus 5.5 (1M context) <noreply@anthropic.com>
Claude-Session: https://claude.ai/code/session_01K3DS9Lp5DvbMPN1T6z91y9
Parts:
- added C125, C126, C127: 100nF 16V X7R, Capacitor_SMD:C_0402_1005Metric, symbol Device:C
- added C128: 10uF 10V X5R, Capacitor_SMD:C_0603_1608Metric, symbol Device:C
- added R133, R134: 2.2k, Resistor_SMD:R_0402_1005Metric, symbol Device:R
- added R135: 100k, Resistor_SMD:R_0402_1005Metric, symbol Device:R
- added R136, R137: 4.7k, Resistor_SMD:R_0402_1005Metric, symbol Device:R
- added U110: SE050E2HQ1/Z01Z3Z, radio:NXP_HX2QFN-20-1EP_3x3mm_P0.4mm_EP1.9x1.9mm, symbol radio:SE050_HX2QFN20
- added U111: LIS3DHTR, Package_LGA:LGA-16_3x3mm_P0.5mm_LayoutBorder3x5y, symbol Sensor_Motion:LIS3DH
Connections:
- net +3V3: now also C125.1, C127.1, C128.1, R133.1, R134.1, R136.1, R137.1, U110.12 (VIN), U111.1 (VDD_IO), U111.14 (VDD), U111.8 (CS)
- net GND: now also C125.2, C126.2, C127.2, C128.2, R135.2, U110.1 (ISO14443_LB), U110.14 (ISO7816_RST_N), U110.17 (ISO14443_LA), U110.19 (VSS), U110.21 (EP), U111.10 (GND), U111.12 (GND), U111.5 (GND), U111.7 (SDO)
- new net ACC_INT1: U111.11 (INT1)
- new net ACC_SCL: R137.2, U111.4 (SPC)
- new net ACC_SDA: R136.2, U111.6 (SDI)
- new net SE_ENA: R135.1, U110.11 (ENA)
- new net SE_SCL: R134.2, U110.10 (I2C_SCL)
- new net SE_SDA: R133.2, U110.9 (I2C_SDA)
- new net SE_VCC: C126.1, U110.15 (VOUT), U110.18 (VCC)
- no-connect marks 23 -> 39
